Commit message: added collisions

File: camera_mount.urdf (robot description, URDF)
Before this commit: robot scene, 6 links, 5 joints
Links:
- link pickup: geometry collision box size=0.23 0.11 0.01; visual box size=0.23 0.11 0.01

File: pi_arm.urdf (robot description, URDF)
Before this commit: robot xArm, 7 links, 6 joints
Links:
- link link5: geometry collision cylinder length=0.004 radius=0.01; visual cylinder length=0.004 radius=0.01
